Commit message: right arm limits

File: src/pybullet_helpers/assets/urdf/human/right_arm_6dof_continuous.urdf (robot description, URDF)
Before this commit: robot right_arm, 9 links, 8 joints
Joints:
- joint base_x: limit (none) -> lower=-1.57 upper=1.57 effort=100 velocity=5.0
- joint base_y: limit (none) -> lower=-0.25 upper=1.57 effort=100 velocity=5.0
- joint base_z: limit (none) -> lower=-1.57 upper=0.25 effort=100 velocity=5.0
- joint lower_to_hand: limit (none) -> lower=-2.0944 upper=0.25 effort=100 velocity=5.0
- joint lower_to_hand_x: limit (none) -> lower=-2.0944 upper=0.25 effort=100 velocity=5.0
- joint upper_to_lower: limit (none) -> lower=-2.0944 upper=0.25 effort=100 velocity=5.0
