Commit message: sneak

File: src/pybullet_helpers/assets/urdf/human/right_arm_7dof_continuous.urdf (robot description, URDF)
Before this commit: robot right_arm, 10 links, 9 joints
Joints:
- joint hand_y_to_hand: limit lower=-2.0944 upper=1.0 effort=100 velocity=5.0 -> lower=-3.14 upper=1.0 effort=100 velocity=5.0
