Commit message: wip

File: src/pybullet_helpers/assets/urdf/human/torso_and_head.urdf (robot description, URDF)
Before this commit: robot torso_and_head, 1 links, 0 joints
Links:
- link base_link: geometry collision mesh filename=meshes/rotated_torso_and_head.stl scale=1.0 1.0 1.0; visual mesh filename=meshes/rotated_torso_and_head.stl scale=1.0 1.0 1.0
