Commit message: add back panda joint limits

File: src/pybullet_helpers/assets/urdf/panda_limb_repo/panda_limb_repo.urdf (robot description, URDF)
Before this commit: robot panda, 12 links, 11 joints
Joints:
- joint panda_joint1: axis 0.0 0.0 1.0 -> 0 0 1; limit (none) -> lower=-2.9671 upper=2.9671 effort= velocity=2.1750; type continuous -> revolute
- joint panda_joint2: axis 0.0 0.0 1.0 -> 0 0 1; limit (none) -> lower=-1.8326 upper=1.8326 effort=87 velocity=2.1750; type continuous -> revolute
- joint panda_joint4: axis 0.0 0.0 1.0 -> 0 0 1; limit (none) -> lower=-3.1416 upper=0.0 effort=87 velocity=2.1750; type continuous -> revolute
- joint panda_joint5: axis 0.0 0.0 1.0 -> 0 0 1; limit (none) -> lower=-2.9671 upper=2.9671 effort=12 velocity=2.6100; type continuous -> revolute
- joint panda_joint6: axis 0.0 0.0 1.0 -> 0 0 1; limit (none) -> lower=-0.0873 upper=3.8223 effort=12 velocity=2.6100; type continuous -> revolute
- joint panda_joint7: axis 0.0 0.0 1.0 -> 0 0 1; limit (none) -> lower=-2.9671 upper=2.9671 effort=12 velocity=2.6100; type continuous -> revolute
