Commit message: change two link robot

File: src/pybullet_helpers/assets/urdf/two_link/two_link_robot.urdf (robot description, URDF)
Before this commit: robot two_link_robot, 4 links, 3 joints
Links:
- link link1: mass 1.0 -> 1; geometry collision box size=1 0.1 0.1; visual box size=1 0.1 0.1
- link link2: mass 1.0 -> 1; geometry collision box size=1 0.1 0.1; visual box size=1 0.1 0.1
Joints:
- joint end_effector: origin xyz=0.5 0 0 rpy=0 1.5708 0 -> xyz=1.0 0 0 rpy=0 1.5708 0
- joint joint1: limit (none) -> lower=-3.14 upper=3.14 effort=1000 velocity=1; origin xyz=0 0 0.1 rpy=0 0 0 -> xyz=0 0 0 rpy=0 0 0; type continuous -> revolute
- joint joint2: axis 0 1 0 -> 0 0 1; limit lower=-0.5 upper=0.5 effort=10.0 velocity=1.0 -> lower=-3.14 upper=3.14 effort=1000 velocity=1; origin xyz=0.0 0 0.5 rpy=0 0 0 -> xyz=1 0 0 rpy=0 0 0

Commit message: fix physics

File: src/pybullet_helpers/assets/urdf/two_link/two_link_robot.urdf (robot description, URDF)
Before this commit: robot two_link_robot, 4 links, 3 joints
Joints:
- joint end_effector: origin xyz=1.0 0 0 rpy=0 1.5708 0 -> xyz=1.0 0 0 rpy=1.5708 0 1.5708
