Commit message: wip

File: src/pybullet_helpers/assets/urdf/kortex_description/gen3_7dof.urdf (robot description, URDF)
Before this commit: robot gen3_robotiq_2f_85, 24 links, 23 joints
Links:
- removed link base_link
- added link my_base_link, mass 1.697; collision mesh filename=package://kortex_description/arms/gen3/7dof/meshes/base_lin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; visual mesh filename=package://kortex_description/arms/gen3/7dof/meshes/base_lin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
Joints:
- joint joint_1: parent base_link -> my_base_link
- joint world_to_root: child base_link -> my_base_link

Commit message: wip

File: src/pybullet_helpers/assets/urdf/kortex_description/gen3_7dof.urdf (robot description, URDF)
Before this commit: robot gen3_robotiq_2f_85, 24 links, 23 joints
Links:
- removed link my_base_link
- added link base_link, mass 1.697; collision mesh filename=package://kortex_description/arms/gen3/7dof/meshes/base_lin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; visual mesh filename=package://kortex_description/arms/gen3/7dof/meshes/base_lin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
Joints:
- joint joint_1: parent my_base_link -> base_link
- joint world_to_root: child my_base_link -> base_link
