Commit message: mesh

File: src/pybullet_helpers/assets/urdf/human_description/human.urdf (robot description, URDF)
Before this commit: robot assistive-human-extracted, 76 links, 75 joints
Links:
- link link10: geometry collision sphere radius=0.89; visual mesh filename=package://head_female_male/BaseHeadMeshes_v5_male_cropped_r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 scale=0.89 0.89 0.89

Commit message: wip

File: src/pybullet_helpers/assets/urdf/human_description/human.urdf (robot description, URDF)
Before this commit: robot assistive-human-extracted, 76 links, 75 joints
Links:
- link link10: geometry collision sphere radius=0.1; visual mesh filename=package://head_female_male/BaseHeadMeshes_v5_male_cropped_r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 scale=0.89 0.89 0.89
Joints:
- joint end_effector: origin xyz=0 0 -0.35 rpy=3.1415926535 0 0 -> xyz=0 0 -0.4 rpy=3.1415926535 0 0

Commit message: wip

File: src/pybullet_helpers/assets/urdf/human_description/human.urdf (robot description, URDF)
Before this commit: robot assistive-human-extracted, 76 links, 75 joints
Links:
- link link10: geometry collision mesh filename=package://head_female_male/BaseHeadMeshes_v5_male_cropped_r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 scale=0.89 0.89 0.89; visual mesh filename=package://head_female_male/BaseHeadMeshes_v5_male_cropped_r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 scale=0.89 0.89 0.89

Commit message: wip

File: src/pybullet_helpers/assets/urdf/human_description/human.urdf (robot description, URDF)
Before this commit: robot assistive-human-extracted, 76 links, 75 joints
Joints:
- joint end_effector: origin xyz=0 0 -0.4 rpy=3.1415926535 0 0 -> xyz=0 0 -0.4 rpy=3.1415926535 0 1.5707963267948966

Commit message: updates to assistive human URDF (#91)

File: src/pybullet_helpers/assets/urdf/human_description/human.urdf (robot description, URDF)
Before this commit: robot assistive-human-extracted, 76 links, 75 joints
Links:
- link link10: geometry collision mesh filename=package://head_female_male/BaseHeadMeshes_v5_male_cropped_r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 scale=0.89 0.89 0.89; visual mesh filename=package://head_female_male/BaseHeadMeshes_v5_male_cropped_r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 scale=0.89 0.89 0.89
Joints:
- joint end_effector: origin xyz=0 0 -0.35 rpy=3.1415926535 0 0 -> xyz=0 0 -0.4 rpy=3.1415926535 0 1.5707963267948966

Commit message: wip

File: src/pybullet_helpers/assets/urdf/human_description/human.urdf (robot description, URDF)
Before this commit: robot assistive-human-extracted, 76 links, 75 joints
Joints:
- joint joint1: limit lower=-0.17453292519943295 upper=0.17453292519943295 effort=0.0 velocity=0.0 -> lower=-0.01 upper=0.01 effort=0.0 velocity=0.0
- joint joint11: limit lower=0.08726646259971647 upper=3.4557519189487724 effort=0.0 velocity=0.0 -> lower=0.08726646259971647 upper=0.75 effort=0.0 velocity=0.0
- joint joint2: limit lower=-0.17453292519943295 upper=0.5235987755982988 effort=0.0 velocity=0.0 -> lower=-0.01 upper=0.01 effort=0.0 velocity=0.0
- joint joint3: limit lower=-0.6108652381980153 upper=0.6108652381980153 effort=0.0 velocity=0.0 -> lower=-0.01 upper=0.01 effort=0.0 velocity=0.0

Commit message: wip

File: src/pybullet_helpers/assets/urdf/human_description/human.urdf (robot description, URDF)
Before this commit: robot assistive-human-extracted, 76 links, 75 joints
Joints:
- joint joint1: limit lower=-0.01 upper=0.01 effort=0.0 velocity=0.0 -> lower=-0.17453292519943295 upper=0.17453292519943295 effort=0.0 velocity=0.0
- joint joint11: limit lower=0.08726646259971647 upper=0.75 effort=0.0 velocity=0.0 -> lower=0.08726646259971647 upper=3.4557519189487724 effort=0.0 velocity=0.0
- joint joint2: limit lower=-0.01 upper=0.01 effort=0.0 velocity=0.0 -> lower=-0.17453292519943295 upper=0.5235987755982988 effort=0.0 velocity=0.0
- joint joint3: limit lower=-0.01 upper=0.01 effort=0.0 velocity=0.0 -> lower=-0.6108652381980153 upper=0.6108652381980153 effort=0.0 velocity=0.0
