Commit message: wip

File: src/pybullet_helpers/assets/urdf/spot/spot.urdf (robot description, URDF)
Before this commit: robot spot, 25 links, 24 joints
Joints:
- joint fl_hx: type revolute -> fixed
- joint fl_hy: type revolute -> fixed
- joint fl_kn: type revolute -> fixed
- joint fr_hx: type revolute -> fixed
- joint fr_hy: type revolute -> fixed
- joint fr_kn: type revolute -> fixed
- joint hl_hx: type revolute -> fixed
- joint hl_hy: type revolute -> fixed
- joint hl_kn: type revolute -> fixed
- joint hr_hx: type revolute -> fixed
- joint hr_hy: type revolute -> fixed
- joint hr_kn: type revolute -> fixed

Commit message: wip

File: src/pybullet_helpers/assets/urdf/spot/spot.urdf (robot description, URDF)
Before this commit: robot spot, 25 links, 24 joints
Joints:
- joint fl_hx: type fixed -> revolute
- joint fl_hy: type fixed -> revolute
- joint fl_kn: type fixed -> revolute
- joint fr_hx: type fixed -> revolute
- joint fr_hy: type fixed -> revolute
- joint fr_kn: type fixed -> revolute
- joint hl_hx: type fixed -> revolute
- joint hl_hy: type fixed -> revolute
- joint hl_kn: type fixed -> revolute
- joint hr_hx: type fixed -> revolute
- joint hr_hy: type fixed -> revolute
- joint hr_kn: type fixed -> revolute

Commit message: change spot end effector frame

File: src/pybullet_helpers/assets/urdf/spot/spot.urdf (robot description, URDF)
Before this commit: robot spot, 25 links, 24 joints
Joints:
- joint hand_frame_joint: origin xyz=0.19557 0.0 0.0 rpy=0 0 0 -> xyz=0.19557 0.0 0.0 rpy=0 1.5707963267948966 0
